Commit message: updates

File: maze_robot_description/urdf/maze_robot.xacro (robot description, xacro)
@@ -108,5 +108,5 @@
   <parent link="base_link"/>
   <child link="right_wheel_1"/>
-  <axis xyz="0.0 -1.0 0.0"/>
+  <axis xyz="0.0 1.0 0.0"/>
 </joint>
 <joint name="left_joint" type="continuous">
